Commit message: add scale in urdf

File: urdf/exoedu_scale.urdf (robot description, URDF)
Before this commit: robot balance, 10 links, 9 joints
Links:
- link lower_arm: geometry visual mesh filename=urdf/EduExo_STL_files/Lower_Arm_Segment.stl scale=0.01 0.01 0.01
- link motor: geometry visual box size=0.40 0.20 0.20
- link motor_adapter: geometry visual mesh filename=urdf/EduExo_STL_files/MotorAdapter.stl scale=0.01 0.01 0.01
- link motor_extend: geometry visual box size=0.10 0.20 0.15
- link sensor: geometry visual box size=0.80 0.20 0.15
- link sensor_adapter: geometry visual mesh filename=urdf/EduExo_STL_files/Interface_Motor_Sensor.stl scale=0.01 0.01 0.01
- link upper_arm: geometry visual mesh filename=urdf/EduExo_STL_files/Upper_Arm_Segment.stl scale=0.01 0.01 0.01
- link upper_cuff0: geometry visual mesh filename=urdf/EduExo_STL_files/EduExoCuffs/Upper_Arm_Cuff_70.stl scale=0.01 0.01 0.01
- link upper_cuff1: geometry visual mesh filename=urdf/EduExo_STL_files/EduExoCuffs/Upper_Arm_Cuff_70.stl scale=0.01 0.01 0.01
Joints:
- joint adapter_upper_joint: origin xyz=25 12 0 rpy=0 0 0 -> xyz=0.25 0.12 0 rpy=0 0 0
- joint arm_cuff0: origin xyz=30 5 -5 rpy=0 0 0 -> xyz=0.30 0.05 -0.05 rpy=0 0 0
- joint arm_cuff1: origin xyz=120 5 -5 rpy=0 0 0 -> xyz=1.20 0.05 -0.05 rpy=0 0 0
- joint base_motor: origin xyz=-5 0 30 rpy=-1.57 0 0 -> xyz=-0.05 0 0.3 rpy=-1.57 0 0
- joint motor_adapter: origin xyz=0 -7 -30 rpy=0 0 0 -> xyz=0 -0.07 -0.3 rpy=0 0 0
- joint motor_extendJoint: origin xyz=-25 0 5 rpy=0 0 0 -> xyz=-0.25 0 0.05 rpy=0 0 0
- joint motor_sensorAdapter: origin xyz=0 0 -10 rpy=0 0 0 -> xyz=0 0 -0.10 rpy=0 0 0
- joint sensorAdapter_sensor: origin xyz=-102 0 -5 rpy=0 0 0 -> xyz=-1.02 0 -0.05 rpy=0 0 0

File: urdf/exoedu_webot.urdf (robot description, URDF)
Before this commit: robot balance, 10 links, 9 joints
Links:
- link lower_arm: geometry visual mesh filename=EduExo_STL_files/Lower_Arm_Segment.stl scale=0.01 0.01 0.01
- link motor: geometry visual box size=0.40 0.20 0.20
- link motor_adapter: geometry visual mesh filename=EduExo_STL_files/MotorAdapter.stl scale=0.01 0.01 0.01
- link motor_extend: geometry visual box size=0.10 0.20 0.15
- link sensor: geometry visual box size=0.80 0.20 0.15
- link sensor_adapter: geometry visual mesh filename=EduExo_STL_files/Interface_Motor_Sensor.stl scale=0.01 0.01 0.01
- link upper_arm: geometry visual mesh filename=EduExo_STL_files/Upper_Arm_Segment.stl scale=0.01 0.01 0.01
- link upper_cuff0: geometry visual mesh filename=EduExo_STL_files/EduExoCuffs/Upper_Arm_Cuff_70.stl scale=0.01 0.01 0.01
- link upper_cuff1: geometry visual mesh filename=EduExo_STL_files/EduExoCuffs/Upper_Arm_Cuff_70.stl scale=0.01 0.01 0.01
Joints:
- joint adapter_upper_joint: origin xyz=25 12 0 rpy=0 0 0 -> xyz=0.25 0.12 0 rpy=0 0 0
- joint arm_cuff0: origin xyz=30 5 -5 rpy=0 0 0 -> xyz=0.30 0.05 -0.05 rpy=0 0 0
- joint arm_cuff1: origin xyz=120 5 -5 rpy=0 0 0 -> xyz=1.20 0.05 -0.05 rpy=0 0 0
- joint base_motor: origin xyz=-5 0 30 rpy=-1.57 0 0 -> xyz=-0.05 0 0.3 rpy=-1.57 0 0
- joint motor_adapter: origin xyz=0 -7 -30 rpy=0 0 0 -> xyz=0 -0.07 -0.3 rpy=0 0 0
- joint motor_extendJoint: origin xyz=-25 0 5 rpy=0 0 0 -> xyz=-0.25 0 0.05 rpy=0 0 0
- joint motor_sensorAdapter: origin xyz=0 0 -10 rpy=0 0 0 -> xyz=0 0 -0.10 rpy=0 0 0
- joint sensorAdapter_sensor: origin xyz=-102 0 -5 rpy=0 0 0 -> xyz=-1.02 0 -0.05 rpy=0 0 0
