Commit message: add ros listener

File: urdf/exoedu_assemble.urdf (robot description, URDF)
Before this commit: robot omnipointer, 10 links, 9 joints
Links:
- removed link upper_cuff0
- removed link upper_cuff1
Joints:
- removed joint arm_cuff0
- removed joint arm_cuff1

Commit message: fix urdf error

File: urdf/exoedu_assemble.urdf (robot description, URDF)
Before this commit: robot balance, 8 links, 7 joints
Links:
- added link upper_cuff0; visual mesh filename=urdf/EduExo_STL_files/EduExoCuffs/Upper_Arm_Cuff_70.stl
- added link upper_cuff1; visual mesh filename=urdf/EduExo_STL_files/EduExoCuffs/Upper_Arm_Cuff_70.stl
Joints:
- added joint arm_cuff0: type fixed, parent upper_arm, child upper_cuff0, origin xyz=30 5 -5 rpy=0 0 0, axis 1 0 0
- added joint arm_cuff1: type fixed, parent upper_arm, child upper_cuff1, origin xyz=120 5 -5 rpy=0 0 0, axis 1 0 0

Commit message: add rm

File: urdf/exoedu_assemble.urdf (robot description, URDF)
Before this commit: robot balance, 10 links, 9 joints
Joints:
- joint base_motor: origin xyz=-5 0 30 rpy=1.57 0 0 -> xyz=-5 0 30 rpy=-1.57 0 0

Commit message: update

File: urdf/exoedu_assemble.urdf (robot description, URDF)
Before this commit: robot balance, 10 links, 9 joints
Links:
- link motor_adapter: geometry visual mesh filename=urdf/EduExo_STL_files/MotorAdapter.stl

File: urdf/exoedu_scale.urdf (robot description, URDF)
Before this commit: robot balance, 10 links, 9 joints
Links:
- link lower_arm: geometry visual mesh filename=urdf/EduExo_STL_files/Lower_Arm_Segment.stl scale=0.005 0.005 0.005
- link motor: geometry visual box size=0.20 0.10 0.10
- link motor_adapter: geometry visual mesh filename=urdf/EduExo_STL_files/MotorAdapter.stl scale=0.005 0.005 0.005
- link motor_extend: geometry visual box size=0.05 0.10 0.075
- link sensor: geometry visual box size=0.40 0.10 0.075
- link sensor_adapter: geometry visual mesh filename=urdf/EduExo_STL_files/Interface_Motor_Sensor.stl scale=0.005 0.005 0.005
- link upper_arm: geometry visual mesh filename=urdf/EduExo_STL_files/Upper_Arm_Segment.stl scale=0.005 0.005 0.005
- link upper_cuff0: geometry visual mesh filename=urdf/EduExo_STL_files/EduExoCuffs/Upper_Arm_Cuff_70.stl scale=0.005 0.005 0.005
- link upper_cuff1: geometry visual mesh filename=urdf/EduExo_STL_files/EduExoCuffs/Upper_Arm_Cuff_70.stl scale=0.005 0.005 0.005
Joints:
- joint adapter_upper_joint: origin xyz=0.25 0.12 0 rpy=0 0 0 -> xyz=0.125 0.06 0 rpy=0 0 0
- joint arm_cuff0: origin xyz=0.30 0.05 -0.05 rpy=0 0 0 -> xyz=0.15 0.025 -0.025 rpy=0 0 0
- joint arm_cuff1: origin xyz=1.20 0.05 -0.05 rpy=0 0 0 -> xyz=0.60 0.025 -0.025 rpy=0 0 0
- joint base_motor: origin xyz=-0.05 0 0.3 rpy=-1.57 0 0 -> xyz=-0.025 0 0.15 rpy=-1.57 0 0
- joint motor_adapter: origin xyz=0 -0.07 -0.3 rpy=0 0 0 -> xyz=0 -0.035 -0.15 rpy=0 0 0
- joint motor_extendJoint: origin xyz=-0.25 0 0.05 rpy=0 0 0 -> xyz=-0.125 0 0.025 rpy=0 0 0
- joint motor_sensorAdapter: origin xyz=0 0 -0.10 rpy=0 0 0 -> xyz=0 0 -0.05 rpy=0 0 0
- joint sensorAdapter_sensor: origin xyz=-1.02 0 -0.05 rpy=0 0 0 -> xyz=-0.51 0 -0.025 rpy=0 0 0
